Commit message: cne

File: src/holosoma/holosoma/data/motions/g1_29dof/whole_body_tracking/objects_largebox.urdf (robot description, URDF)
Before this commit: robot largebox.urdf, 1 links, 0 joints
Links:
- link baseLink: geometry collision box size=0.47115421 0.45873013 0.40789548; visual mesh filename=largebox.obj scale=1.0 1.0 1.0

Commit message: behave

File: src/holosoma/holosoma/data/motions/g1_29dof/whole_body_tracking/objects_largebox.urdf (robot description, URDF)
Before this commit: robot largebox.urdf, 1 links, 0 joints
Links:
- link baseLink: geometry collision mesh filename=largebox.obj scale=1.0 1.0 1.0; visual mesh filename=largebox.obj scale=1.0 1.0 1.0
