Commit message: fix-multi-train-bug

File: logs/sim2sim_exports/object_urdfs/box_10__box_10__eff10__motion_size_box_collision.urdf (robot description, URDF)
Before this commit: robot box_74__eff09_box_collision, 1 links, 0 joints
Links:
- link baseLink: geometry collision box size=0.4585590958595276 0.2551282048225403 0.22102713584899902; visual mesh filename=/home/ubuntu/FAR/holosoma/data/ds_box_data/scale_mix_all/tr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 scale=1 1 1
