Commit message: added

File: logs/sim2sim_exports/object_urdfs/box_74__box_74__baseline__motion_size_box_collision.urdf (robot description, URDF)
Before this commit: robot box_10_box_collision, 1 links, 0 joints
Links:
- link baseLink: geometry collision box size=0.46575260162353516 0.42469602823257446 0.24985061585903168; visual mesh filename=/home/ubuntu/FAR/holosoma/data/ds_box_data/scale_mix_all/tr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 scale=1.32193955 1.32193957 1.32193953

File: logs/sim2sim_exports/object_urdfs/box_74__box_74__motion_size_box_collision.urdf (robot description, URDF)
Before this commit: robot box_74_box_collision, 1 links, 0 joints
Links:
- link baseLink: geometry collision box size=0.46575260162353516 0.42469602823257446 0.24985061585903168; visual mesh filename=/home/ubuntu/FAR/holosoma/data/ds_box_data/train_g1_w_obj_p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 scale=1.32193954 1.32193956 1.32193952

File: logs/sim2sim_exports/object_urdfs/box_75__box_75__motion_size_box_collision.urdf (robot description, URDF)
Before this commit: robot box_75_box_collision, 1 links, 0 joints
Links:
- link baseLink: geometry collision box size=0.3469197750091553 0.3472353219985962 0.3352038562297821; visual mesh filename=/home/ubuntu/FAR/holosoma/data/ds_box_data/train_g1_w_obj_p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 scale=1.23958695 1.23958697 1.23958695
