Commit message: added

File: logs/sim2sim_exports/object_urdfs/box_100__baseline__box_100__baseline__motion_size_box_collision.urdf (robot description, URDF)
Before this commit: robot box_74_box_collision, 1 links, 0 joints
Links:
- link baseLink: geometry collision box size=0.38682061433792114 0.21348148584365845 0.1884974092245102; visual mesh filename=/home/ubuntu/FAR/holosoma/data/ds_box_data/scale_mix_all/tr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 scale=1 1 1

File: logs/sim2sim_exports/object_urdfs/box_200__baseline__box_200__baseline__motion_size_box_collision.urdf (robot description, URDF)
Before this commit: robot box_74_box_collision, 1 links, 0 joints
Links:
- link baseLink: geometry collision box size=0.47870489954948425 0.26419124007225037 0.2332724630832672; visual mesh filename=/home/ubuntu/FAR/holosoma/data/ds_box_data/scale_mix_all/tr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 scale=1 1 1

File: logs/sim2sim_exports/object_urdfs/box_401__baseline__box_401__baseline__motion_size_box_collision.urdf (robot description, URDF)
Before this commit: robot box_74_box_collision, 1 links, 0 joints
Links:
- link baseLink: geometry collision box size=0.37315547466278076 0.20593984425067902 0.18183837831020355; visual mesh filename=/home/ubuntu/FAR/holosoma/data/ds_box_data/scale_mix_all/tr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 scale=1 1 1
