Commit message: mocap works

File: logs/sim2sim_exports/object_urdfs/box_10__box_10__motion_size_box_collision.urdf (robot description, URDF)
Before this commit: robot box_74_box_collision, 1 links, 0 joints
Links:
- link baseLink: geometry collision box size=0.4585590958595276 0.2551282048225403 0.22102713584899902; visual mesh filename=/home/ubuntu/FAR/holosoma/data/ds_box_data_legacy/train_g1_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 scale=1.28587889 1.28587893 1.28587888

File: logs/sim2sim_exports/object_urdfs/box_10__box_10__urdf_size_box_collision.urdf (robot description, URDF)
Before this commit: robot box_74_box_collision, 1 links, 0 joints
Links:
- link baseLink: geometry collision box size=0.356611418 0.1984076404 0.1718879894; visual mesh filename=/home/ubuntu/FAR/holosoma/data/ds_box_data_legacy/train_g1_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 scale=1 1 1

File: logs/sim2sim_exports/object_urdfs/box_74__box_74__eff09__urdf_size_box_collision.urdf (robot description, URDF)
Before this commit: robot box_74_box_collision, 1 links, 0 joints
Links:
- link baseLink: geometry collision box size=0.419177328 0.382226408 0.224865552; visual mesh filename=/home/ubuntu/FAR/holosoma/data/ds_box_data/scale_mix_all/tr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 scale=1 1 1

File: logs/sim2sim_exports/object_urdfs/box_74__box_74__motion_size.urdf (robot description, URDF)
Before this commit: robot box_74_box_collision, 1 links, 0 joints
Links:
- link baseLink: geometry collision mesh filename=/home/ubuntu/FAR/holosoma/data/ds_box_data_legacy/train_g1_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 scale=1.32193954 1.32193956 1.32193952; visual mesh filename=/home/ubuntu/FAR/holosoma/data/ds_box_data_legacy/train_g1_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 scale=1.32193954 1.32193956 1.32193952

File: logs/sim2sim_exports/object_urdfs/box_74__box_74__urdf_size_box_collision.urdf (robot description, URDF)
Before this commit: robot box_74_box_collision, 1 links, 0 joints
Links:
- link baseLink: geometry collision box size=0.352325192 0.321267356 0.1890030618; visual mesh filename=/home/ubuntu/FAR/holosoma/data/ds_box_data_legacy/train_g1_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 scale=1 1 1

File: logs/sim2sim_exports/object_urdfs/box_75__box_75__motion_size_box_collision.urdf (robot description, URDF)
Before this commit: robot box_74_box_collision, 1 links, 0 joints
Links:
- link baseLink: geometry collision box size=0.3469197750091553 0.3472353219985962 0.3352038562297821; visual mesh filename=/home/ubuntu/FAR/holosoma/data/ds_box_data_legacy/train_g1_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 scale=1.23958695 1.23958697 1.23958695

File: logs/sim2sim_exports/object_urdfs/box_75__box_75__urdf_size_box_collision.urdf (robot description, URDF)
Before this commit: robot box_74_box_collision, 1 links, 0 joints
Links:
- link baseLink: geometry collision box size=0.279867238 0.280121792 0.270415768; visual mesh filename=/home/ubuntu/FAR/holosoma/data/ds_box_data_legacy/train_g1_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 scale=1 1 1

Commit message: added

File: logs/sim2sim_exports/object_urdfs/box_10__box_10__motion_size_box_collision.urdf (robot description, URDF)
Before this commit: robot box_10_box_collision, 1 links, 0 joints
Links:
- link baseLink: geometry collision box size=0.4585590958595276 0.2551282048225403 0.22102713584899902; visual mesh filename=/home/ubuntu/FAR/holosoma/data/ds_box_data_legacy/train_g1_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 scale=1.28587889 1.28587893 1.28587888

File: logs/sim2sim_exports/object_urdfs/box_75__box_75__motion_size_box_collision.urdf (robot description, URDF)
Before this commit: robot box_75_box_collision, 1 links, 0 joints
Links:
- link baseLink: geometry collision box size=0.3469197750091553 0.3472353219985962 0.3352038562297821; visual mesh filename=/home/ubuntu/FAR/holosoma/data/ds_box_data_legacy/train_g1_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 scale=1.23958695 1.23958697 1.23958695
