Commit message: Restore MuJoCo box rollout defaults

File: data_demo/objects/box_74.urdf (robot description, URDF)
Before this commit: robot box_74, 1 links, 0 joints
Links:
- link baseLink: geometry collision box size=0.46575260162353516 0.42469602823257446 0.24985061585903168; visual mesh filename=box_74.obj scale=1.32193954 1.32193956 1.32193952

File: data_demo/objects/box_75.urdf (robot description, URDF)
Before this commit: robot box_75, 1 links, 0 joints
Links:
- link baseLink: geometry collision box size=0.3469197750091553 0.3472353219985962 0.3352038562297821; visual mesh filename=box_75.obj scale=1.23958695 1.23958697 1.23958695
